File: circuit/Atari 5200 Controller Port Emulator.brd (EAGLE design)
At the start: 50.8 x 40.6 mm, 24 parts, among them IC1 PIC16F628P

Commit message: Corrected TXD/RXD connections to RX232 module header
Connections:
- removed net RX-IN: IC1.7, SV1.4
- removed net TX-OUT: IC1.8, SV1.3
- new net RXI: IC1.8, SV1.4
- new net TXD: IC1.7, SV1.3
Routing:
- net TXD: track 0.00 -> 46.9 mm
- net TX-OUT: track 41.7 -> 0.00 mm
- net RX-IN: track 39.0 -> 0.00 mm
- net RXI: track 0.00 -> 35.3 mm
Changed lines of the file:
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@@
 <?xml version="1.0" encoding="utf-8"?>
 <!DOCTYPE eagle SYSTEM "eagle.dtd">
-<eagle version="7.2.0">
+<eagle version="7.3.0">
 <drawing>
 <settings>
@@
 <layers>
 <layer number="1" name="Top" color="4" fill="1" visible="no" active="yes"/>
-<layer number="16" name="Bottom" color="1" fill="1" visible="no" active="yes"/>
+<layer number="16" name="Bottom" color="1" fill="1" visible="yes" active="yes"/>
 <layer number="17" name="Pads" color="2" fill="1" visible="yes" active="yes"/>
 <layer number="18" name="Vias" color="2" fill="1" visible="yes" active="yes"/>
@@
 <wire x1="28.575" y1="16.51" x2="26.67" y2="16.51" width="0.3048" layer="16"/>
 </signal>
-<signal name="RX-IN">
-<contactref element="IC1" pad="7"/>
+<signal name="RXI">
 <contactref element="SV1" pad="4"/>
 <wire x1="5.715" y1="21.59" x2="3.81" y2="21.59" width="0.3048" layer="16"/>
@@
 <wire x1="3.175" y1="22.225" x2="3.175" y2="32.385" width="0.3048" layer="16"/>
 <wire x1="3.175" y1="32.385" x2="8.89" y2="38.1" width="0.3048" layer="16"/>
-<wire x1="8.89" y1="38.1" x2="16.51" y2="38.1" width="0.3048" layer="16"/>
-<wire x1="16.51" y1="38.1" x2="17.78" y2="36.83" width="0.3048" layer="16"/>
-<wire x1="17.78" y1="36.83" x2="17.78" y2="32.385" width="0.3048" layer="16"/>
-<wire x1="17.78" y1="32.385" x2="18.415" y2="31.75" width="0.3048" layer="16"/>
-<wire x1="18.415" y1="31.75" x2="21.59" y2="31.75" width="0.3048" layer="16"/>
-</signal>
-<signal name="TX-OUT">
+<wire x1="8.89" y1="38.1" x2="15.875" y2="38.1" width="0.3048" layer="16"/>
+<wire x1="15.875" y1="38.1" x2="19.685" y2="34.29" width="0.3048" layer="16"/>
 <contactref element="IC1" pad="8"/>
+<wire x1="19.685" y1="34.29" x2="21.59" y2="34.29" width="0.3048" layer="16"/>
+</signal>
+<signal name="TXD">
 <contactref element="SV1" pad="3"/>
-<wire x1="21.59" y1="34.29" x2="19.685" y2="34.29" width="0.3048" layer="16"/>
-<wire x1="19.685" y1="34.29" x2="19.05" y2="34.925" width="0.3048" layer="16"/>
-<wire x1="19.05" y1="34.925" x2="19.05" y2="36.83" width="0.3048" layer="16"/>
-<wire x1="19.05" y1="36.83" x2="17.145" y2="38.735" width="0.3048" layer="16"/>
-<wire x1="17.145" y1="38.735" x2="8.255" y2="38.735" width="0.3048" layer="16"/>
+<wire x1="19.685" y1="35.56" x2="16.51" y2="38.735" width="0.3048" layer="16"/>
+<wire x1="16.51" y1="38.735" x2="8.255" y2="38.735" width="0.3048" layer="16"/>
 <wire x1="8.255" y1="38.735" x2="1.905" y2="32.385" width="0.3048" layer="16"/>
 <wire x1="1.905" y1="32.385" x2="1.905" y2="20.32" width="0.3048" layer="16"/>
 <wire x1="1.905" y1="20.32" x2="3.175" y2="19.05" width="0.3048" layer="16"/>
 <wire x1="3.175" y1="19.05" x2="5.715" y2="19.05" width="0.3048" layer="16"/>
+<contactref element="IC1" pad="7"/>
+<wire x1="19.685" y1="35.56" x2="22.86" y2="35.56" width="0.3048" layer="16"/>
+<wire x1="22.86" y1="35.56" x2="23.495" y2="34.925" width="0.3048" layer="16"/>
+<wire x1="23.495" y1="34.925" x2="23.495" y2="32.385" width="0.3048" layer="16"/>
+<wire x1="23.495" y1="32.385" x2="22.86" y2="31.75" width="0.3048" layer="16"/>
+<wire x1="22.86" y1="31.75" x2="21.59" y2="31.75" width="0.3048" layer="16"/>
 </signal>
 <signal name="TOP/VPP">
