File: circuit/Atari 5200 Controller Port Emulator.brd (EAGLE design)
At the start: 50.8 x 40.6 mm, 22 parts, among them IC1 PIC16F628P

Commit message: Keyboard scan OK, buttons OK, Pot reading works but need validation
Parts:
- added C6: 100n, rcl:C050-024X044
- added R14: 1k, rcl:0204/7
Connections:
- net GND: now also C6.2, R14.2
- net VPOT: now also C6.1, R14.1
Routing:
- net VPOT: track 39.9 -> 65.0 mm
- net LINE0: track 35.7 -> 20.8 mm
- net LINE2: track 13.8 -> 20.1 mm
- net LINE1: track 13.8 -> 17.6 mm
- net +5V: track 88.8 -> 85.3 mm
- net POTX: track 21.0 -> 22.8 mm
- net LINE3: track 39.5 -> 38.2 mm

Commit message: Updated schematics
Connections:
- net BOTTOM renamed TOP
- net TOP/VPP renamed BOT/VPP
Changed lines of the file:
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@@
 <grid distance="0.025" unitdist="inch" unit="inch" style="dots" multiple="2" display="yes" altdistance="0.0125" altunitdist="inch" altunit="inch"/>
 <layers>
-<layer number="1" name="Top" color="4" fill="1" visible="no" active="yes"/>
-<layer number="16" name="Bottom" color="1" fill="1" visible="no" active="yes"/>
+<layer number="1" name="Top" color="4" fill="1" visible="yes" active="yes"/>
+<layer number="16" name="Bottom" color="1" fill="1" visible="yes" active="yes"/>
 <layer number="17" name="Pads" color="2" fill="1" visible="yes" active="yes"/>
 <layer number="18" name="Vias" color="2" fill="1" visible="yes" active="yes"/>
@@
 <wire x1="3.175" y1="19.05" x2="5.715" y2="19.05" width="0.3048" layer="16"/>
 </signal>
-<signal name="TOP/VPP">
+<signal name="BOT/VPP">
 <contactref element="IC1" pad="4"/>
 <contactref element="R11" pad="2"/>
@@
 <wire x1="42.3164" y1="25.8064" x2="43.18" y2="26.67" width="0.3048" layer="16"/>
 </signal>
-<signal name="BOTTOM">
+<signal name="TOP">
 <contactref element="IC1" pad="9"/>
 <contactref element="R12" pad="1"/>

Commit message: Working version, updated schematics
Parts:
- turned R11 to 180 degrees
Connections:
- net RX-IN renamed TXD
- net TX-OUT renamed RXI
- net BOT/VPP: now also R12.1; no longer R13.1
- net TOP: now also R13.1; no longer R12.1
Routing:
- net BOT/VPP: track 40.0 -> 32.2 mm
- net TOP: track 8.67 -> 15.8 mm
- net TXD: track 39.0 -> 33.5 mm
- net +5V: track 85.3 -> 81.5 mm
- net RXI: track 41.7 -> 38.4 mm
Changed lines of the file:
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@@
 <grid distance="0.025" unitdist="inch" unit="inch" style="dots" multiple="2" display="yes" altdistance="0.0125" altunitdist="inch" altunit="inch"/>
 <layers>
-<layer number="1" name="Top" color="4" fill="1" visible="yes" active="yes"/>
+<layer number="1" name="Top" color="4" fill="1" visible="no" active="yes"/>
 <layer number="16" name="Bottom" color="1" fill="1" visible="yes" active="yes"/>
 <layer number="17" name="Pads" color="2" fill="1" visible="yes" active="yes"/>
@@
 <attribute name="VALUE" x="29.4894" y="8.4074" size="0.9906" layer="27" ratio="10"/>
 </element>
-<element name="R11" library="rcl" package="0204/7" value="47k" x="30.48" y="34.29" smashed="yes">
+<element name="R11" library="rcl" package="0204/7" value="47k" x="30.48" y="34.29" smashed="yes" rot="R180">
 <attribute name="NAME" x="26.035" y="34.8996" size="1.016" layer="25" ratio="10" rot="R180"/>
 <attribute name="VALUE" x="29.4894" y="33.8074" size="1.016" layer="27" ratio="10"/>
@@
 <contactref element="R11" pad="1"/>
 <contactref element="SV2" pad="2"/>
-<wire x1="26.67" y1="34.29" x2="30.48" y2="34.29" width="0.4064" layer="1"/>
-<wire x1="30.48" y1="34.29" x2="32.385" y2="32.385" width="0.4064" layer="1"/>
+<wire x1="34.29" y1="34.29" x2="32.385" y2="32.385" width="0.4064" layer="1"/>
 <wire x1="32.385" y1="32.385" x2="32.385" y2="20.32" width="0.4064" layer="1"/>
 <wire x1="32.385" y1="20.32" x2="31.115" y2="19.05" width="0.4064" layer="1"/>
@@
 <wire x1="28.575" y1="16.51" x2="26.67" y2="16.51" width="0.3048" layer="16"/>
 </signal>
-<signal name="RX-IN">
-<contactref element="IC1" pad="7"/>
-<contactref element="SV1" pad="4"/>
-<wire x1="5.715" y1="21.59" x2="3.81" y2="21.59" width="0.3048" layer="16"/>
-<wire x1="3.81" y1="21.59" x2="3.175" y2="22.225" width="0.3048" layer="16"/>
-<wire x1="3.175" y1="22.225" x2="3.175" y2="32.385" width="0.3048" layer="16"/>
-<wire x1="3.175" y1="32.385" x2="8.89" y2="38.1" width="0.3048" layer="16"/>
-<wire x1="8.89" y1="38.1" x2="16.51" y2="38.1" width="0.3048" layer="16"/>
-<wire x1="16.51" y1="38.1" x2="17.78" y2="36.83" width="0.3048" layer="16"/>
-<wire x1="17.78" y1="36.83" x2="17.78" y2="32.385" width="0.3048" layer="16"/>
-<wire x1="17.78" y1="32.385" x2="18.415" y2="31.75" width="0.3048" layer="16"/>
-<wire x1="18.415" y1="31.75" x2="21.59" y2="31.75" width="0.3048" layer="16"/>
-</signal>
-<signal name="TX-OUT">
-<contactref element="IC1" pad="8"/>
-<contactref element="SV1" pad="3"/>
-<wire x1="21.59" y1="34.29" x2="19.685" y2="34.29" width="0.3048" layer="16"/>
-<wire x1="19.685" y1="34.29" x2="19.05" y2="34.925" width="0.3048" layer="16"/>
-<wire x1="19.05" y1="34.925" x2="19.05" y2="36.83" width="0.3048" layer="16"/>
-<wire x1="19.05" y1="36.83" x2="17.145" y2="38.735" width="0.3048" layer="16"/>
-<wire x1="17.145" y1="38.735" x2="8.255" y2="38.735" width="0.3048" layer="16"/>
-<wire x1="8.255" y1="38.735" x2="1.905" y2="32.385" width="0.3048" layer="16"/>
-<wire x1="1.905" y1="32.385" x2="1.905" y2="20.32" width="0.3048" layer="16"/>
-<wire x1="1.905" y1="20.32" x2="3.175" y2="19.05" width="0.3048" layer="16"/>
-<wire x1="3.175" y1="19.05" x2="5.715" y2="19.05" width="0.3048" layer="16"/>
-</signal>
 <signal name="BOT/VPP">
-<contactref element="IC1" pad="4"/>
-<contactref element="R11" pad="2"/>
-<contactref element="R13" pad="1"/>
 <contactref element="SV2" pad="1"/>
-<wire x1="26.67" y1="29.21" x2="29.21" y2="29.21" width="0.3048" layer="16"/>
-<wire x1="29.21" y1="29.21" x2="30.48" y2="30.48" width="0.3048" layer="16"/>
-<wire x1="30.48" y1="30.48" x2="30.48" y2="33.02" width="0.3048" layer="16"/>
-<wire x1="30.48" y1="33.02" x2="31.75" y2="34.29" width="0.3048" layer="16"/>
-<wire x1="31.75" y1="34.29" x2="34.29" y2="34.29" width="0.3048" layer="16"/>
 <wire x1="10.16" y1="21.59" x2="10.795" y2="21.59" width="0.3048" layer="16"/>
 <wire x1="10.795" y1="21.59" x2="12.065" y2="22.86" width="0.3048" layer="16"/>
@@
 <wire x1="12.7" y1="25.4" x2="17.78" y2="25.4" width="0.3048" layer="16"/>
 <wire x1="17.78" y1="25.4" x2="19.05" y2="24.13" width="0.3048" layer="16"/>
-<wire x1="19.05" y1="24.13" x2="21.59" y2="24.13" width="0.3048" layer="16"/>
-<wire x1="26.67" y1="29.21" x2="26.035" y2="29.21" width="0.3048" layer="16"/>
-<wire x1="26.035" y1="29.21" x2="24.765" y2="30.48" width="0.3048" layer="16"/>
-<wire x1="24.765" y1="30.48" x2="18.415" y2="30.48" width="0.3048" layer="16"/>
+<wire x1="24.13" y1="30.48" x2="18.415" y2="30.48" width="0.3048" layer="16"/>
 <wire x1="18.415" y1="30.48" x2="17.78" y2="29.845" width="0.3048" layer="16"/>
 <wire x1="17.78" y1="29.845" x2="17.78" y2="25.4" width="0.3048" layer="16"/>
+<contactref element="R12" pad="1"/>
+<contactref element="R11" pad="2"/>
+<contactref element="IC1" pad="4"/>
+<wire x1="19.05" y1="24.13" x2="21.59" y2="24.13" width="0.3048" layer="16"/>
+<wire x1="26.67" y1="31.75" x2="25.4" y2="31.75" width="0.3048" layer="16"/>
+<wire x1="25.4" y1="31.75" x2="24.13" y2="30.48" width="0.3048" layer="16"/>
+<wire x1="26.67" y1="34.29" x2="26.035" y2="34.29" width="0.3048" layer="16"/>
+<wire x1="26.035" y1="34.29" x2="25.4" y2="33.655" width="0.3048" layer="16"/>
+<wire x1="25.4" y1="33.655" x2="25.4" y2="31.75" width="0.3048" layer="16"/>
 </signal>
 <signal name="B">
@@
 <wire x1="42.3164" y1="25.8064" x2="43.18" y2="26.67" width="0.3048" layer="16"/>
 </signal>
+<signal name="TXD">
+<contactref element="IC1" pad="7"/>
+<contactref element="SV1" pad="4"/>
+<wire x1="5.715" y1="21.59" x2="3.81" y2="21.59" width="0.3048" layer="16"/>
+<wire x1="3.81" y1="21.59" x2="3.175" y2="22.225" width="0.3048" layer="16"/>
+<wire x1="3.175" y1="22.225" x2="3.175" y2="31.115" width="0.3048" layer="16"/>
+<wire x1="3.175" y1="31.115" x2="7.62" y2="35.56" width="0.3048" layer="16"/>
+<wire x1="7.62" y1="35.56" x2="15.24" y2="35.56" width="0.3048" layer="16"/>
+<wire x1="15.24" y1="35.56" x2="19.05" y2="31.75" width="0.3048" layer="16"/>
+<wire x1="19.05" y1="31.75" x2="21.59" y2="31.75" width="0.3048" layer="16"/>
+</signal>
+<signal name="RXI">
+<contactref element="IC1" pad="8"/>
+<contactref element="SV1" pad="3"/>
+<wire x1="21.59" y1="34.29" x2="19.685" y2="34.29" width="0.3048" layer="16"/>
+<wire x1="19.685" y1="34.29" x2="15.875" y2="38.1" width="0.3048" layer="16"/>
+<wire x1="15.875" y1="38.1" x2="8.89" y2="38.1" width="0.3048" layer="16"/>
+<wire x1="8.89" y1="38.1" x2="2.54" y2="31.75" width="0.3048" layer="16"/>
+<wire x1="2.54" y1="31.75" x2="2.54" y2="20.32" width="0.3048" layer="16"/>
+<wire x1="2.54" y1="20.32" x2="3.81" y2="19.05" width="0.3048" layer="16"/>
+<wire x1="3.81" y1="19.05" x2="5.715" y2="19.05" width="0.3048" layer="16"/>
+</signal>
 <signal name="TOP">
+<contactref element="R13" pad="1"/>
 <contactref element="IC1" pad="9"/>
-<contactref element="R12" pad="1"/>
-<wire x1="21.59" y1="36.83" x2="24.13" y2="36.83" width="0.3048" layer="16"/>
-<wire x1="24.13" y1="36.83" x2="24.765" y2="36.195" width="0.3048" layer="16"/>
-<wire x1="24.765" y1="36.195" x2="24.765" y2="33.655" width="0.3048" layer="16"/>
-<wire x1="24.765" y1="33.655" x2="26.67" y2="31.75" width="0.3048" layer="16"/>
+<wire x1="21.59" y1="36.83" x2="27.94" y2="36.83" width="0.3048" layer="16"/>
+<wire x1="27.94" y1="36.83" x2="28.575" y2="36.195" width="0.3048" layer="16"/>
+<wire x1="28.575" y1="36.195" x2="28.575" y2="29.845" width="0.3048" layer="16"/>
+<wire x1="28.575" y1="29.845" x2="27.94" y2="29.21" width="0.3048" layer="16"/>
+<wire x1="27.94" y1="29.21" x2="26.67" y2="29.21" width="0.3048" layer="16"/>
 </signal>
 </signals>
