File: circuit/Atari 5200 Controller Port Emulator.sch (EAGLE design)
At the start: 22 parts, among them IC1 PIC16F628P

Commit message: Keyboard scan OK, buttons OK, Pot reading works but need validation
Parts:
- added C6: 100n, rcl:C-EU050-024X044
- added R14: 1k, rcl:R-EU_0204/7
Connections:
- net GND: now also C6.2, R14.2
- net VPOT: now also C6.1, R14.1
Changed lines of the file:
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@@
 <part name="SV1" library="con-lstb" deviceset="MA06-1" device="" value="SERIAL"/>
 <part name="SV2" library="con-lstb" deviceset="MA06-1" device="" value="PGM"/>
+<part name="C6" library="rcl" deviceset="C-EU" device="050-024X044" value="100n"/>
+<part name="R14" library="rcl" deviceset="R-EU_" device="0204/7" value="1k"/>
+<part name="GND8" library="supply1" deviceset="GND" device=""/>
 </parts>
 <sheets>
@@
 </instance>
 <instance part="P+1" gate="1" x="172.72" y="88.9" smashed="yes" rot="R270">
-<attribute name="VALUE" x="172.72" y="86.36" size="1.778" layer="96"/>
+<attribute name="VALUE" x="177.038" y="90.678" size="1.778" layer="96" rot="R180"/>
 </instance>
 <instance part="P+2" gate="1" x="33.02" y="104.14"/>
@@
 <instance part="SV1" gate="1" x="10.16" y="81.28" rot="MR180"/>
 <instance part="SV2" gate="1" x="38.1" y="20.32" rot="MR180"/>
+<instance part="C6" gate="G$1" x="165.1" y="78.74" smashed="yes" rot="MR0">
+<attribute name="NAME" x="166.624" y="80.899" size="1.778" layer="95" rot="MR180"/>
+<attribute name="VALUE" x="166.624" y="73.279" size="1.778" layer="96" rot="MR180"/>
+</instance>
+<instance part="R14" gate="G$1" x="154.94" y="76.2" smashed="yes" rot="MR270">
+<attribute name="NAME" x="156.718" y="79.0194" size="1.778" layer="95" rot="MR180"/>
+<attribute name="VALUE" x="156.718" y="76.2" size="1.778" layer="96" rot="MR180"/>
+</instance>
+<instance part="GND8" gate="1" x="154.94" y="66.04" rot="MR0"/>
 </instances>
 <busses>
@@
 <label x="48.26" y="22.86" size="1.778" layer="95"/>
 </segment>
+<segment>
+<pinref part="C6" gate="G$1" pin="2"/>
+<pinref part="GND8" gate="1" pin="GND"/>
+<pinref part="R14" gate="G$1" pin="2"/>
+<wire x1="154.94" y1="71.12" x2="154.94" y2="68.58" width="0.1524" layer="91"/>
+<junction x="154.94" y="71.12"/>
+<wire x1="154.94" y1="71.12" x2="165.1" y2="71.12" width="0.1524" layer="91"/>
+<wire x1="165.1" y1="71.12" x2="165.1" y2="73.66" width="0.1524" layer="91"/>
+</segment>
 </net>
 <net name="LF/RG" class="0">
@@
 <wire x1="147.32" y1="60.96" x2="152.4" y2="60.96" width="0.1524" layer="91"/>
 <pinref part="X1" gate="-1" pin="10"/>
-<wire x1="147.32" y1="83.82" x2="157.48" y2="83.82" width="0.1524" layer="91"/>
-<wire x1="157.48" y1="83.82" x2="157.48" y2="60.96" width="0.1524" layer="91"/>
-<wire x1="157.48" y1="60.96" x2="152.4" y2="60.96" width="0.1524" layer="91"/>
+<wire x1="147.32" y1="83.82" x2="172.72" y2="83.82" width="0.1524" layer="91"/>
+<wire x1="172.72" y1="83.82" x2="172.72" y2="60.96" width="0.1524" layer="91"/>
+<wire x1="172.72" y1="60.96" x2="152.4" y2="60.96" width="0.1524" layer="91"/>
 <junction x="152.4" y="60.96"/>
 <label x="147.32" y="83.82" size="1.778" layer="95"/>
@@
 <wire x1="147.32" y1="43.18" x2="152.4" y2="43.18" width="0.1524" layer="91"/>
 <pinref part="X1" gate="-1" pin="11"/>
-<wire x1="147.32" y1="86.36" x2="160.02" y2="86.36" width="0.1524" layer="91"/>
-<wire x1="160.02" y1="86.36" x2="160.02" y2="43.18" width="0.1524" layer="91"/>
-<wire x1="160.02" y1="43.18" x2="152.4" y2="43.18" width="0.1524" layer="91"/>
+<wire x1="147.32" y1="86.36" x2="175.26" y2="86.36" width="0.1524" layer="91"/>
+<wire x1="175.26" y1="86.36" x2="175.26" y2="43.18" width="0.1524" layer="91"/>
+<wire x1="175.26" y1="43.18" x2="152.4" y2="43.18" width="0.1524" layer="91"/>
 <junction x="152.4" y="43.18"/>
 <label x="147.32" y="86.36" size="1.778" layer="95"/>
@@
 <wire x1="76.2" y1="81.28" x2="101.6" y2="81.28" width="0.1524" layer="91"/>
 <wire x1="101.6" y1="81.28" x2="101.6" y2="71.12" width="0.1524" layer="91"/>
-<wire x1="101.6" y1="71.12" x2="154.94" y2="71.12" width="0.1524" layer="91"/>
-<wire x1="154.94" y1="71.12" x2="154.94" y2="81.28" width="0.1524" layer="91"/>
+<wire x1="101.6" y1="71.12" x2="149.86" y2="71.12" width="0.1524" layer="91"/>
+<label x="78.74" y="81.28" size="1.778" layer="95"/>
 <pinref part="X1" gate="-1" pin="9"/>
-<wire x1="154.94" y1="81.28" x2="147.32" y2="81.28" width="0.1524" layer="91"/>
-<label x="78.74" y="81.28" size="1.778" layer="95"/>
+<wire x1="149.86" y1="81.28" x2="147.32" y2="81.28" width="0.1524" layer="91"/>
+<pinref part="R14" gate="G$1" pin="1"/>
 <label x="147.32" y="81.28" size="1.778" layer="95"/>
-</segment>
-</net>
+<wire x1="149.86" y1="71.12" x2="149.86" y2="81.28" width="0.1524" layer="91"/>
+<junction x="149.86" y="81.28"/>
+<pinref part="C6" gate="G$1" pin="1"/>
+<wire x1="149.86" y1="81.28" x2="154.94" y2="81.28" width="0.1524" layer="91"/>
+<wire x1="154.94" y1="81.28" x2="165.1" y2="81.28" width="0.1524" layer="91"/>
+<junction x="154.94" y="81.28"/>
+</segment>
+</net>

Commit message: Corrected TXD/RXD connections to RX232 module header
Connections:
- removed net RX-IN: IC1.RB1/RX/DT, SV1.4
- removed net TX-OUT: IC1.RB2/TX/CK, SV1.3
- new net RXI: IC1.RB2/TX/CK, SV1.4
- new net TXD: IC1.RB1/RX/DT, SV1.3
Changed lines of the file:
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@@
 <?xml version="1.0" encoding="utf-8"?>
 <!DOCTYPE eagle SYSTEM "eagle.dtd">
-<eagle version="7.2.0">
+<eagle version="7.3.0">
 <drawing>
 <settings>
@@
 </segment>
 </net>
-<net name="RX-IN" class="0">
-<segment>
-<pinref part="IC1" gate="G$1" pin="RB1/RX/DT"/>
-<wire x1="76.2" y1="83.82" x2="88.9" y2="83.82" width="0.1524" layer="91"/>
-<wire x1="88.9" y1="83.82" x2="88.9" y2="40.64" width="0.1524" layer="91"/>
-<wire x1="88.9" y1="40.64" x2="25.4" y2="40.64" width="0.1524" layer="91"/>
+<net name="RXI" class="0">
+<segment>
+<wire x1="76.2" y1="86.36" x2="91.44" y2="86.36" width="0.1524" layer="91"/>
+<wire x1="91.44" y1="86.36" x2="91.44" y2="40.64" width="0.1524" layer="91"/>
+<wire x1="91.44" y1="40.64" x2="25.4" y2="40.64" width="0.1524" layer="91"/>
 <wire x1="25.4" y1="40.64" x2="25.4" y2="81.28" width="0.1524" layer="91"/>
 <wire x1="25.4" y1="81.28" x2="17.78" y2="81.28" width="0.1524" layer="91"/>
-<label x="78.74" y="83.82" size="1.778" layer="95"/>
+<label x="78.74" y="86.36" size="1.778" layer="95"/>
 <pinref part="SV1" gate="1" pin="4"/>
 <label x="20.32" y="81.28" size="1.778" layer="95"/>
-</segment>
-</net>
-<net name="TX-OUT" class="0">
-<segment>
 <pinref part="IC1" gate="G$1" pin="RB2/TX/CK"/>
-<wire x1="76.2" y1="86.36" x2="91.44" y2="86.36" width="0.1524" layer="91"/>
-<wire x1="91.44" y1="86.36" x2="91.44" y2="38.1" width="0.1524" layer="91"/>
-<wire x1="91.44" y1="38.1" x2="27.94" y2="38.1" width="0.1524" layer="91"/>
-<wire x1="27.94" y1="38.1" x2="27.94" y2="83.82" width="0.1524" layer="91"/>
+</segment>
+</net>
+<net name="TXD" class="0">
+<segment>
+<wire x1="76.2" y1="83.82" x2="88.9" y2="83.82" width="0.1524" layer="91"/>
+<wire x1="88.9" y1="83.82" x2="88.9" y2="43.18" width="0.1524" layer="91"/>
+<wire x1="88.9" y1="43.18" x2="27.94" y2="43.18" width="0.1524" layer="91"/>
+<wire x1="27.94" y1="43.18" x2="27.94" y2="83.82" width="0.1524" layer="91"/>
 <wire x1="27.94" y1="83.82" x2="17.78" y2="83.82" width="0.1524" layer="91"/>
-<label x="78.74" y="86.36" size="1.778" layer="95"/>
+<label x="78.74" y="83.82" size="1.778" layer="95"/>
 <pinref part="SV1" gate="1" pin="3"/>
 <label x="20.32" y="83.82" size="1.778" layer="95"/>
-</segment>
-</net>
+<pinref part="IC1" gate="G$1" pin="RB1/RX/DT"/>
+</segment>
+</net>
