File: circuit/Atari 5200 Controller Port Emulator.sch (EAGLE design)
At the start: 24 parts, among them IC1 PIC16F628P

Commit message: Updated schematics
Connections:
- net BOTTOM renamed TOP
- net TOP/VPP renamed BOT/VPP
Changed lines of the file:
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@@
 </segment>
 </net>
-<net name="TOP/VPP" class="0">
+<net name="BOT/VPP" class="0">
 <segment>
 <pinref part="IC1" gate="G$1" pin="RA5/MCLR/VPP"/>
@@
 </segment>
 </net>
-<net name="BOTTOM" class="0">
+<net name="TOP" class="0">
 <segment>
 <pinref part="IC1" gate="G$1" pin="RB3/CCP1"/>
